File: hw/board/pwr_board.sch (EAGLE design)
At the start: 65 parts, among them IC1 7805T

Commit message: separation in two boards - work in progress
Parts:
- removed J1, J2: (no value), SparkFun-Connectors:M14
- removed JP1: (no value), SparkFun-RF:XBEE-1B1
- removed JP5: DNP, SparkFun-Connectors:M05PTH
- removed JP6: DNP, SparkFun-Connectors:M03PTH
- removed LB, LF, RB, RF, TO_PWRBRD_SINGNALS: (no value), SparkFun-Connectors:M03X2POGO_PINS
- removed LED1, LED2: Red, SparkFun-LED:LED-RED0603
- removed LED3, LED4, LED5: Green, SparkFun-LED:LED-GREEN0603
- removed R1, R11, R2, R3, R4: 1k, SparkFun-Resistors:1KOHM1/10W1%(0603)
- removed S3: Reset, SparkFun-Electromechanical:SWITCH-MOMENTARY-2SMD
- removed TO_PWRBRD_PWR, VIN: (no value), con-wago-500:W237-102
- removed U$1: TEENSY_3.0_ALL_PINS, Teensy_3_and_LC_Series_Boards_v1.1:TEENSY_3.0_ALL_PINS
Connections:
- removed net 3.3V: J2.2, JP1.VDD, JP5.2, R1.1, R11.2, R3.1, U$1.3.3V
- removed net A14/DAC: JP5.5, U$1.RESET
- removed net CHARGE: J1.5, TO_PWRBRD_SINGNALS.5, U$1.8
- removed net CHIP: J1.2, TO_PWRBRD_SINGNALS.6, U$1.11
- removed net CTS: JP1.CTS
- removed net DIO0: JP1.DIO0
- removed net DIO1: JP1.DIO1
- removed net DIO11: JP1.DIO11
- removed net DIO12: JP1.DIO12
- removed net DIO2: JP1.DIO2
- removed net DIO3: JP1.DIO3
- removed net DIO4: JP1.DIO4
- removed net DIO5: JP1.DIO5, R2.2
- removed net DIO9: JP1.DIO9
- removed net DISCHARGE: J1.4, U$1.9
- removed net DRIBBLE: J1.3, TO_PWRBRD_SINGNALS.4, U$1.10
- removed net DTR: JP1.DTR
- removed net LBBRK: J1.6, LB.4, U$1.7
- removed net LBDIR: J1.7, LB.3, U$1.6
- removed net LBENA: J1.8, LB.2, U$1.5
- removed net LBSPEED: J2.5, LB.5, U$1.22/A8
- removed net LFBRK: J1.9, LF.4, U$1.4
- removed net LFDIR: J1.10, LF.3, U$1.3
- removed net LFENA: J1.11, LF.2, U$1.2
- removed net LFSPEED: J2.4, LF.5, U$1.23/A9
- removed net N$1: J1.1, U$1.12
- removed net N$12: LED1.A, R11.1
- removed net N$139: LED5.A, R2.1
- removed net N$17: LED2.A, R1.2
- removed net N$18: J2.3, U$1.AGND
- removed net N$19: LED3.A, R3.2
- removed net N$43: LED4.A, R4.1
- removed net P13: J2.14, U$1.13
- removed net PROG: JP5.4, U$1.PGM
- removed net PWR_GND: CAPACITOR-2.KL, T3.E, TO_UPVOLT-2.KL, U$2.EMITTER, U$4.P$4, UP-VOLT_REG-1.KL
- removed net PWR_VCC: C4.1, LM338.IN, TO_UPVOLT-1.KL
- removed net RBBRK: J2.13, RB.4, U$1.14/A0
- removed net RBDIR: J2.12, RB.3, U$1.15/A1
- removed net RBENA: J2.11, RB.2, U$1.16/A2
- removed net RBSPEED: J2.7, RB.5, U$1.20/A6
- removed net READ_250: TO_PWRBRD_SINGNALS.1, U$1.A11
- removed net READ_CAP: TO_PWRBRD_SINGNALS.3, U$1.A10
- removed net RES: JP1.RES@8
- removed net RES2: JP1.RES@14
- removed net RESET: JP1.RESET, S3.1
- removed net RFBRK: J2.10, RF.4, U$1.17/A3
- removed net RFDIR: J2.9, RF.3, U$1.18/A4
- removed net RFENA: J2.8, RF.2, U$1.19/A5
- removed net RFSPEED: J2.6, RF.5, U$1.21/A7
- removed net RSSI: JP1.RSSI, R4.2
- removed net RTS: JP1.RTS
- removed net UART_RX: J1.13, JP1.DOUT, LED2.C, U$1.0
- removed net UART_TX: J1.12, JP1.DIN, LED3.C, U$1.1
- removed net VBAT: JP5.1, U$1.VBAT
- new net GND_PWR: CAPACITOR-2.KL, PWR_PWR_IN-2.KL, U$2.EMITTER, UP-VOLT_REG-1.KL
- new net VCC: C1.1, C4.1, IC1.VI, LM338.IN, PWR_PWR_IN-1.KL, TO_UPVOLT-1.KL
- net +24V: no longer C1.1, IC1.VI, TO_PWRBRD_PWR-1.KL, VIN-1.KL
- net +5V: no longer U$1.VIN
- net GND: now also T3.E, TO_UPVOLT-2.KL, U$4.P$4; no longer J1.14, JP1.GND, JP5.3, JP6.1, JP6.2, JP6.3, LB.1, LED1.C, LED4.C, LED5.C, LF.1, RB.1, RF.1, S3.2, TO_PWRBRD_PWR-2.KL, U$1.GND, VIN-2.KL
Other:
- note removed: "Controllers"
- note removed: "LEDs"
- note removed: "Teensy 3.2"
- note removed: "XBee"
- moved on the sheet: C1, C2, CAPACITOR-1, IC1, PWR_PWR_IN-1, PWR_PWR_IN-2
